Commit message: Decide singularity, tip-over and overload on their own ontology ids.
The projector used to fold these into PHY.JOINT_LIMIT. Mirror the checks in the Python fallback and make the 22-row gold set actually trip them.

File: dataset/urdf/panda_arm_simple.urdf (robot description, URDF)
Before this commit: robot panda_arm_simple, 7 links, 6 joints
Links:
- added link panda_link6
Joints:
- added joint panda_joint7: type revolute, parent panda_link6, child panda_hand, origin xyz=0.088 0 0 rpy=1.5707963267948966 0 0, axis 0 0 1, limit lower=-2.8973 upper=2.8973 effort=12 velocity=2.610
- joint panda_joint6: child panda_hand -> panda_link6
